File: schematic/Unit_LTP305G/Unit_LTP305G.kicad_pcb (KiCad board)
At the start: 2 copper layers, 58.9 x 20.6 mm, 10 parts, among them J1 Conn_01x04, U1 M5StampS3, U2 LTP305G

Commit message: schematic
Parts:
- moved J1 0.26 mm to (165.7, 67.9)
